Commit message: Modify moveit packages to work with pandaX_-joints and links.

File: panda1_moveit_config/config/hand.xacro (robot description, xacro)
@@ -8,9 +8,9 @@
     <!--SUBGROUPS: Groups can also be formed by referencing to already defined group names-->
     <group name="hand">
-      <link name="panda_hand" />
-      <link name="panda_leftfinger" />
-      <link name="panda_rightfinger" />
-      <joint name="panda_finger_joint1" />
-      <passive_joint name="panda_finger_joint2" />
+      <link name="panda1_hand" />
+      <link name="panda1_leftfinger" />
+      <link name="panda1_rightfinger" />
+      <joint name="panda1_finger_joint1" />
+      <passive_joint name="panda1_finger_joint2" />
       <!--link name="panda_tcp" />
       <passive_joint name="panda_hand_tcp_joint" /-->
@@ -19,7 +19,7 @@
     <!--END EFFECTOR: Purpose: Represent information about an end effector.-->
     <!--DISABLE COLLISIONS: By default it is assumed that any link of the robot could potentially come into collision with any other link in the robot. This tag disables collision checking between a specified pair of links. -->
-    <disable_collisions link1="panda_hand" link2="panda_leftfinger" reason="Adjacent" />
-    <disable_collisions link1="panda_hand" link2="panda_rightfinger" reason="Adjacent" />
-    <disable_collisions link1="panda_leftfinger" link2="panda_rightfinger" reason="Default" />
+    <disable_collisions link1="panda1_hand" link2="panda1_leftfinger" reason="Adjacent" />
+    <disable_collisions link1="panda1_hand" link2="panda1_rightfinger" reason="Adjacent" />
+    <disable_collisions link1="panda1_leftfinger" link2="panda1_rightfinger" reason="Default" />
   </xacro:macro>
 </robot>

File: panda1_moveit_config/config/panda_arm.srdf.xacro (robot description, xacro)
@@ -5,5 +5,5 @@
 -->
 <robot xmlns:xacro="http://www.ros.org/wiki/xacro" name="panda">
-  <xacro:include filename="$(find panda_moveit_config)/config/panda_arm.xacro" />
+  <xacro:include filename="$(find panda1_moveit_config)/config/panda_arm.xacro" />
   <xacro:panda_arm />
 </robot>

File: panda1_moveit_config/config/panda_arm.xacro (robot description, xacro)
@@ -8,39 +8,39 @@
     <!--SUBGROUPS: Groups can also be formed by referencing to already defined group names-->
     <group name="panda_arm">
-      <chain base_link="panda_link0" tip_link="panda_link8" />
+      <chain base_link="panda1_link0" tip_link="panda1_link8" />
     </group>
     <!--GROUP STATES: Purpose: Define a named state for a particular group, in terms of joint values. This is useful to define states like 'folded arms'-->
     <group_state name="ready" group="panda_arm">
-      <joint name="panda_joint1" value="0" />
-      <joint name="panda_joint2" value="-0.785" />
-      <joint name="panda_joint3" value="0" />
-      <joint name="panda_joint4" value="-2.356" />
-      <joint name="panda_joint5" value="0" />
-      <joint name="panda_joint6" value="1.571" />
-      <joint name="panda_joint7" value="0.785" />
+      <joint name="panda1_joint1" value="0" />
+      <joint name="panda1_joint2" value="-0.785" />
+      <joint name="panda1_joint3" value="0" />
+      <joint name="panda1_joint4" value="-2.356" />
+      <joint name="panda1_joint5" value="0" />
+      <joint name="panda1_joint6" value="1.571" />
+      <joint name="panda1_joint7" value="0.785" />
     </group_state>
     <!--END EFFECTOR: Purpose: Represent information about an end effector.-->
     <!--VIRTUAL JOINT: Purpose: this element defines a virtual joint between a robot link and an external frame of reference (considered fixed with respect to the robot)-->
-    <virtual_joint name="virtual_joint" type="fixed" parent_frame="world" child_link="panda_link0" />
+    <virtual_joint name="virtual_joint" type="fixed" parent_frame="world" child_link="panda1_link0" />
     <!--DISABLE COLLISIONS: By default it is assumed that any link of the robot could potentially come into collision with any other link in the robot. This tag disables collision checking between a specified pair of links. -->
-    <disable_collisions link1="panda_link0" link2="panda_link1" reason="Adjacent" />
-    <disable_collisions link1="panda_link0" link2="panda_link2" reason="Never" />
-    <disable_collisions link1="panda_link0" link2="panda_link3" reason="Never" />
-    <disable_collisions link1="panda_link0" link2="panda_link4" reason="Never" />
-    <disable_collisions link1="panda_link1" link2="panda_link2" reason="Adjacent" />
-    <disable_collisions link1="panda_link1" link2="panda_link3" reason="Never" />
-    <disable_collisions link1="panda_link1" link2="panda_link4" reason="Never" />
-    <disable_collisions link1="panda_link2" link2="panda_link3" reason="Adjacent" />
-    <disable_collisions link1="panda_link2" link2="panda_link4" reason="Never" />
-    <disable_collisions link1="panda_link2" link2="panda_link6" reason="Never" />
-    <disable_collisions link1="panda_link3" link2="panda_link4" reason="Adjacent" />
-    <disable_collisions link1="panda_link3" link2="panda_link5" reason="Never" />
-    <disable_collisions link1="panda_link3" link2="panda_link6" reason="Never" />
-    <disable_collisions link1="panda_link3" link2="panda_link7" reason="Never" />
-    <disable_collisions link1="panda_link4" link2="panda_link5" reason="Adjacent" />
-    <disable_collisions link1="panda_link4" link2="panda_link6" reason="Never" />
-    <disable_collisions link1="panda_link4" link2="panda_link7" reason="Never" />
-    <disable_collisions link1="panda_link5" link2="panda_link6" reason="Adjacent" />
-    <disable_collisions link1="panda_link6" link2="panda_link7" reason="Adjacent" />
+    <disable_collisions link1="panda1_link0" link2="panda1_link1" reason="Adjacent" />
+    <disable_collisions link1="panda1_link0" link2="panda1_link2" reason="Never" />
+    <disable_collisions link1="panda1_link0" link2="panda1_link3" reason="Never" />
+    <disable_collisions link1="panda1_link0" link2="panda1_link4" reason="Never" />
+    <disable_collisions link1="panda1_link1" link2="panda1_link2" reason="Adjacent" />
+    <disable_collisions link1="panda1_link1" link2="panda1_link3" reason="Never" />
+    <disable_collisions link1="panda1_link1" link2="panda1_link4" reason="Never" />
+    <disable_collisions link1="panda1_link2" link2="panda1_link3" reason="Adjacent" />
+    <disable_collisions link1="panda1_link2" link2="panda1_link4" reason="Never" />
+    <disable_collisions link1="panda1_link2" link2="panda1_link6" reason="Never" />
+    <disable_collisions link1="panda1_link3" link2="panda1_link4" reason="Adjacent" />
+    <disable_collisions link1="panda1_link3" link2="panda1_link5" reason="Never" />
+    <disable_collisions link1="panda1_link3" link2="panda1_link6" reason="Never" />
+    <disable_collisions link1="panda1_link3" link2="panda1_link7" reason="Never" />
+    <disable_collisions link1="panda1_link4" link2="panda1_link5" reason="Adjacent" />
+    <disable_collisions link1="panda1_link4" link2="panda1_link6" reason="Never" />
+    <disable_collisions link1="panda1_link4" link2="panda1_link7" reason="Never" />
+    <disable_collisions link1="panda1_link5" link2="panda1_link6" reason="Adjacent" />
+    <disable_collisions link1="panda1_link6" link2="panda1_link7" reason="Adjacent" />
   </xacro:macro>
 </robot>

File: panda1_moveit_config/config/panda_arm_hand.srdf.xacro (robot description, xacro)
@@ -5,6 +5,6 @@
 -->
 <robot xmlns:xacro="http://www.ros.org/wiki/xacro" name="panda">
-  <xacro:include filename="$(find panda_moveit_config)/config/panda_arm.xacro" />
-  <xacro:include filename="$(find panda_moveit_config)/config/hand.xacro" />
+  <xacro:include filename="$(find panda1_moveit_config)/config/panda_arm.xacro" />
+  <xacro:include filename="$(find panda1_moveit_config)/config/hand.xacro" />
   <xacro:panda_arm />
   <xacro:hand />
@@ -20,26 +20,26 @@
   <!--GROUP STATES: Purpose: Define a named state for a particular group, in terms of joint values. This is useful to define states like 'folded arms'-->
   <group_state name="ready" group="panda_arm_hand">
-    <joint name="panda_joint1" value="0" />
-    <joint name="panda_joint2" value="-0.785" />
-    <joint name="panda_joint3" value="0" />
-    <joint name="panda_joint4" value="-2.356" />
-    <joint name="panda_joint5" value="0" />
-    <joint name="panda_joint6" value="1.571" />
-    <joint name="panda_joint7" value="0.785" />
+    <joint name="panda1_joint1" value="0" />
+    <joint name="panda1_joint2" value="-0.785" />
+    <joint name="panda1_joint3" value="0" />
+    <joint name="panda1_joint4" value="-2.356" />
+    <joint name="panda1_joint5" value="0" />
+    <joint name="panda1_joint6" value="1.571" />
+    <joint name="panda1_joint7" value="0.785" />
   </group_state>
   <!--END EFFECTOR: Purpose: Represent information about an end effector.-->
-  <end_effector name="hand" parent_link="panda_link8" group="hand" parent_group="panda_arm_hand" />
+  <end_effector name="hand" parent_link="panda1_link8" group="hand" parent_group="panda_arm_hand" />
   <!--DISABLE COLLISIONS: By default it is assumed that any link of the robot could potentially come into collision with any other link in the robot. This tag disables collision checking between a specified pair of links. -->
-  <disable_collisions link1="panda_hand" link2="panda_link3" reason="Never" />
-  <disable_collisions link1="panda_hand" link2="panda_link4" reason="Never" />
-  <disable_collisions link1="panda_hand" link2="panda_link6" reason="Never" />
-  <disable_collisions link1="panda_hand" link2="panda_link7" reason="Adjacent" />
-  <disable_collisions link1="panda_leftfinger" link2="panda_link3" reason="Never" />
-  <disable_collisions link1="panda_leftfinger" link2="panda_link4" reason="Never" />
-  <disable_collisions link1="panda_leftfinger" link2="panda_link6" reason="Never" />
-  <disable_collisions link1="panda_leftfinger" link2="panda_link7" reason="Never" />
-  <disable_collisions link1="panda_link3" link2="panda_rightfinger" reason="Never" />
-  <disable_collisions link1="panda_link4" link2="panda_rightfinger" reason="Never" />
-  <disable_collisions link1="panda_link6" link2="panda_rightfinger" reason="Never" />
-  <disable_collisions link1="panda_link7" link2="panda_rightfinger" reason="Never" />
+  <disable_collisions link1="panda1_hand" link2="panda1_link3" reason="Never" />
+  <disable_collisions link1="panda1_hand" link2="panda1_link4" reason="Never" />
+  <disable_collisions link1="panda1_hand" link2="panda1_link6" reason="Never" />
+  <disable_collisions link1="panda1_hand" link2="panda1_link7" reason="Adjacent" />
+  <disable_collisions link1="panda1_leftfinger" link2="panda1_link3" reason="Never" />
+  <disable_collisions link1="panda1_leftfinger" link2="panda1_link4" reason="Never" />
+  <disable_collisions link1="panda1_leftfinger" link2="panda1_link6" reason="Never" />
+  <disable_collisions link1="panda1_leftfinger" link2="panda1_link7" reason="Never" />
+  <disable_collisions link1="panda1_link3" link2="panda1_rightfinger" reason="Never" />
+  <disable_collisions link1="panda1_link4" link2="panda1_rightfinger" reason="Never" />
+  <disable_collisions link1="panda1_link6" link2="panda1_rightfinger" reason="Never" />
+  <disable_collisions link1="panda1_link7" link2="panda1_rightfinger" reason="Never" />
 </robot>

File: panda2_moveit_config/config/hand.xacro (robot description, xacro)
@@ -8,9 +8,9 @@
     <!--SUBGROUPS: Groups can also be formed by referencing to already defined group names-->
     <group name="hand">
-      <link name="panda_hand" />
-      <link name="panda_leftfinger" />
-      <link name="panda_rightfinger" />
-      <joint name="panda_finger_joint1" />
-      <passive_joint name="panda_finger_joint2" />
+      <link name="panda2_hand" />
+      <link name="panda2_leftfinger" />
+      <link name="panda2_rightfinger" />
+      <joint name="panda2_finger_joint1" />
+      <passive_joint name="panda2_finger_joint2" />
       <!--link name="panda_tcp" />
       <passive_joint name="panda_hand_tcp_joint" /-->
@@ -19,7 +19,7 @@
     <!--END EFFECTOR: Purpose: Represent information about an end effector.-->
     <!--DISABLE COLLISIONS: By default it is assumed that any link of the robot could potentially come into collision with any other link in the robot. This tag disables collision checking between a specified pair of links. -->
-    <disable_collisions link1="panda_hand" link2="panda_leftfinger" reason="Adjacent" />
-    <disable_collisions link1="panda_hand" link2="panda_rightfinger" reason="Adjacent" />
-    <disable_collisions link1="panda_leftfinger" link2="panda_rightfinger" reason="Default" />
+    <disable_collisions link1="panda2_hand" link2="panda2_leftfinger" reason="Adjacent" />
+    <disable_collisions link1="panda2_hand" link2="panda2_rightfinger" reason="Adjacent" />
+    <disable_collisions link1="panda2_leftfinger" link2="panda2_rightfinger" reason="Default" />
   </xacro:macro>
 </robot>

File: panda2_moveit_config/config/panda_arm.srdf.xacro (robot description, xacro)
@@ -5,5 +5,5 @@
 -->
 <robot xmlns:xacro="http://www.ros.org/wiki/xacro" name="panda">
-  <xacro:include filename="$(find panda_moveit_config)/config/panda_arm.xacro" />
+  <xacro:include filename="$(find panda2_moveit_config)/config/panda_arm.xacro" />
   <xacro:panda_arm />
 </robot>

File: panda2_moveit_config/config/panda_arm.xacro (robot description, xacro)
@@ -8,39 +8,39 @@
     <!--SUBGROUPS: Groups can also be formed by referencing to already defined group names-->
     <group name="panda_arm">
-      <chain base_link="panda_link0" tip_link="panda_link8" />
+      <chain base_link="panda2_link0" tip_link="panda2_link8" />
     </group>
     <!--GROUP STATES: Purpose: Define a named state for a particular group, in terms of joint values. This is useful to define states like 'folded arms'-->
     <group_state name="ready" group="panda_arm">
-      <joint name="panda_joint1" value="0" />
-      <joint name="panda_joint2" value="-0.785" />
-      <joint name="panda_joint3" value="0" />
-      <joint name="panda_joint4" value="-2.356" />
-      <joint name="panda_joint5" value="0" />
-      <joint name="panda_joint6" value="1.571" />
-      <joint name="panda_joint7" value="0.785" />
+      <joint name="panda2_joint1" value="0" />
+      <joint name="panda2_joint2" value="-0.785" />
+      <joint name="panda2_joint3" value="0" />
+      <joint name="panda2_joint4" value="-2.356" />
+      <joint name="panda2_joint5" value="0" />
+      <joint name="panda2_joint6" value="1.571" />
+      <joint name="panda2_joint7" value="0.785" />
     </group_state>
     <!--END EFFECTOR: Purpose: Represent information about an end effector.-->
     <!--VIRTUAL JOINT: Purpose: this element defines a virtual joint between a robot link and an external frame of reference (considered fixed with respect to the robot)-->
-    <virtual_joint name="virtual_joint" type="fixed" parent_frame="world" child_link="panda_link0" />
+    <virtual_joint name="virtual_joint" type="fixed" parent_frame="world" child_link="panda2_link0" />
     <!--DISABLE COLLISIONS: By default it is assumed that any link of the robot could potentially come into collision with any other link in the robot. This tag disables collision checking between a specified pair of links. -->
-    <disable_collisions link1="panda_link0" link2="panda_link1" reason="Adjacent" />
-    <disable_collisions link1="panda_link0" link2="panda_link2" reason="Never" />
-    <disable_collisions link1="panda_link0" link2="panda_link3" reason="Never" />
-    <disable_collisions link1="panda_link0" link2="panda_link4" reason="Never" />
-    <disable_collisions link1="panda_link1" link2="panda_link2" reason="Adjacent" />
-    <disable_collisions link1="panda_link1" link2="panda_link3" reason="Never" />
-    <disable_collisions link1="panda_link1" link2="panda_link4" reason="Never" />
-    <disable_collisions link1="panda_link2" link2="panda_link3" reason="Adjacent" />
-    <disable_collisions link1="panda_link2" link2="panda_link4" reason="Never" />
-    <disable_collisions link1="panda_link2" link2="panda_link6" reason="Never" />
-    <disable_collisions link1="panda_link3" link2="panda_link4" reason="Adjacent" />
-    <disable_collisions link1="panda_link3" link2="panda_link5" reason="Never" />
-    <disable_collisions link1="panda_link3" link2="panda_link6" reason="Never" />
-    <disable_collisions link1="panda_link3" link2="panda_link7" reason="Never" />
-    <disable_collisions link1="panda_link4" link2="panda_link5" reason="Adjacent" />
-    <disable_collisions link1="panda_link4" link2="panda_link6" reason="Never" />
-    <disable_collisions link1="panda_link4" link2="panda_link7" reason="Never" />
-    <disable_collisions link1="panda_link5" link2="panda_link6" reason="Adjacent" />
-    <disable_collisions link1="panda_link6" link2="panda_link7" reason="Adjacent" />
+    <disable_collisions link1="panda2_link0" link2="panda2_link1" reason="Adjacent" />
+    <disable_collisions link1="panda2_link0" link2="panda2_link2" reason="Never" />
+    <disable_collisions link1="panda2_link0" link2="panda2_link3" reason="Never" />
+    <disable_collisions link1="panda2_link0" link2="panda2_link4" reason="Never" />
+    <disable_collisions link1="panda2_link1" link2="panda2_link2" reason="Adjacent" />
+    <disable_collisions link1="panda2_link1" link2="panda2_link3" reason="Never" />
+    <disable_collisions link1="panda2_link1" link2="panda2_link4" reason="Never" />
+    <disable_collisions link1="panda2_link2" link2="panda2_link3" reason="Adjacent" />
+    <disable_collisions link1="panda2_link2" link2="panda2_link4" reason="Never" />
+    <disable_collisions link1="panda2_link2" link2="panda2_link6" reason="Never" />
+    <disable_collisions link1="panda2_link3" link2="panda2_link4" reason="Adjacent" />
+    <disable_collisions link1="panda2_link3" link2="panda2_link5" reason="Never" />
+    <disable_collisions link1="panda2_link3" link2="panda2_link6" reason="Never" />
+    <disable_collisions link1="panda2_link3" link2="panda2_link7" reason="Never" />
+    <disable_collisions link1="panda2_link4" link2="panda2_link5" reason="Adjacent" />
+    <disable_collisions link1="panda2_link4" link2="panda2_link6" reason="Never" />
+    <disable_collisions link1="panda2_link4" link2="panda2_link7" reason="Never" />
+    <disable_collisions link1="panda2_link5" link2="panda2_link6" reason="Adjacent" />
+    <disable_collisions link1="panda2_link6" link2="panda2_link7" reason="Adjacent" />
   </xacro:macro>
 </robot>

File: panda2_moveit_config/config/panda_arm_hand.srdf.xacro (robot description, xacro)
@@ -5,6 +5,6 @@
 -->
 <robot xmlns:xacro="http://www.ros.org/wiki/xacro" name="panda">
-  <xacro:include filename="$(find panda_moveit_config)/config/panda_arm.xacro" />
-  <xacro:include filename="$(find panda_moveit_config)/config/hand.xacro" />
+  <xacro:include filename="$(find panda2_moveit_config)/config/panda_arm.xacro" />
+  <xacro:include filename="$(find panda2_moveit_config)/config/hand.xacro" />
   <xacro:panda_arm />
   <xacro:hand />
@@ -20,26 +20,26 @@
   <!--GROUP STATES: Purpose: Define a named state for a particular group, in terms of joint values. This is useful to define states like 'folded arms'-->
   <group_state name="ready" group="panda_arm_hand">
-    <joint name="panda_joint1" value="0" />
-    <joint name="panda_joint2" value="-0.785" />
-    <joint name="panda_joint3" value="0" />
-    <joint name="panda_joint4" value="-2.356" />
-    <joint name="panda_joint5" value="0" />
-    <joint name="panda_joint6" value="1.571" />
-    <joint name="panda_joint7" value="0.785" />
+    <joint name="panda2_joint1" value="0" />
+    <joint name="panda2_joint2" value="-0.785" />
+    <joint name="panda2_joint3" value="0" />
+    <joint name="panda2_joint4" value="-2.356" />
+    <joint name="panda2_joint5" value="0" />
+    <joint name="panda2_joint6" value="1.571" />
+    <joint name="panda2_joint7" value="0.785" />
   </group_state>
   <!--END EFFECTOR: Purpose: Represent information about an end effector.-->
-  <end_effector name="hand" parent_link="panda_link8" group="hand" parent_group="panda_arm_hand" />
+  <end_effector name="hand" parent_link="panda2_link8" group="hand" parent_group="panda_arm_hand" />
   <!--DISABLE COLLISIONS: By default it is assumed that any link of the robot could potentially come into collision with any other link in the robot. This tag disables collision checking between a specified pair of links. -->
-  <disable_collisions link1="panda_hand" link2="panda_link3" reason="Never" />
-  <disable_collisions link1="panda_hand" link2="panda_link4" reason="Never" />
-  <disable_collisions link1="panda_hand" link2="panda_link6" reason="Never" />
-  <disable_collisions link1="panda_hand" link2="panda_link7" reason="Adjacent" />
-  <disable_collisions link1="panda_leftfinger" link2="panda_link3" reason="Never" />
-  <disable_collisions link1="panda_leftfinger" link2="panda_link4" reason="Never" />
-  <disable_collisions link1="panda_leftfinger" link2="panda_link6" reason="Never" />
-  <disable_collisions link1="panda_leftfinger" link2="panda_link7" reason="Never" />
-  <disable_collisions link1="panda_link3" link2="panda_rightfinger" reason="Never" />
-  <disable_collisions link1="panda_link4" link2="panda_rightfinger" reason="Never" />
-  <disable_collisions link1="panda_link6" link2="panda_rightfinger" reason="Never" />
-  <disable_collisions link1="panda_link7" link2="panda_rightfinger" reason="Never" />
+  <disable_collisions link1="panda2_hand" link2="panda2_link3" reason="Never" />
+  <disable_collisions link1="panda2_hand" link2="panda2_link4" reason="Never" />
+  <disable_collisions link1="panda2_hand" link2="panda2_link6" reason="Never" />
+  <disable_collisions link1="panda2_hand" link2="panda2_link7" reason="Adjacent" />
+  <disable_collisions link1="panda2_leftfinger" link2="panda2_link3" reason="Never" />
+  <disable_collisions link1="panda2_leftfinger" link2="panda2_link4" reason="Never" />
+  <disable_collisions link1="panda2_leftfinger" link2="panda2_link6" reason="Never" />
+  <disable_collisions link1="panda2_leftfinger" link2="panda2_link7" reason="Never" />
+  <disable_collisions link1="panda2_link3" link2="panda2_rightfinger" reason="Never" />
+  <disable_collisions link1="panda2_link4" link2="panda2_rightfinger" reason="Never" />
+  <disable_collisions link1="panda2_link6" link2="panda2_rightfinger" reason="Never" />
+  <disable_collisions link1="panda2_link7" link2="panda2_rightfinger" reason="Never" />
 </robot>
